File: PCB/knuckle sense pcb v-1/knuckle sense pcb v-1.kicad_sch (KiCad schematic)
At the start: 0 parts

Commit message: COMPLETE
Parts:
- added BT1: Battery_Cell, Battery:BatteryHolder_Keystone_3034_1x20mm, symbol Device:Battery_Cell
- added D1, D2: LED, LED_THT:LED_D5.0mm, symbol Device:LED
- added R1, R2: 1kR, Resistor_THT:R_Axial_DIN0207_L6.3mm_D2.5mm_P7.62mm_Horizontal, symbol Device:R
Connections:
- new net: BT1.1 (+), D1.2 (A), D2.2 (A)
- new net: BT1.2 (-), R1.2, R2.1
- new net: D1.1 (K), R2.2
- new net: D2.1 (K), R1.1
